Commit message: Added walls to environment

File: PathPlanning/data/plane.urdf (robot description, URDF)
Before this commit: robot plane, 1 links, 0 joints
Links:
- added link bottom_wall; collision box size=30 1 1; visual box size=30 1 1
- added link left_wall; collision box size=1 32 1; visual box size=1 32 1
- added link right_wall; collision box size=1 32 1; visual box size=1 32 1
- added link top_wall; collision box size=30 1 1; visual box size=30 1 1
- link planeLink: geometry collision box size=32 32 10; visual mesh filename=plane.obj scale=1 1 1
Joints:
- added joint joint1: type fixed, parent planeLink, child left_wall
- added joint joint2: type fixed, parent planeLink, child right_wall
- added joint joint3: type fixed, parent planeLink, child top_wall
- added joint joint4: type fixed, parent planeLink, child bottom_wall
